Commit message: Filtragem da nuvem de pontos para mostrar só a zona relevante

File: free_space_detection/urdf/atlas2.urdf (robot description, URDF)
Before this commit: robot ATLCASCAR2, 1 links, 0 joints
Links:
- removed link map
- added link moving_axis; visual mesh filename=package://free_space_detection/stl_files/atlas2.STL
