Commit message: Criação de um modulo em python para analisar geometricamente os feixes do laser

File: scan_simulator/urdf/atlas2.urdf.xacro (robot description, xacro)
@@ -21,4 +21,5 @@
     </inertial>
   </link>
+  <!-- Sensores de varrimento 2D -->
   <!-- hokuyo0 -->
   <link name="laser_link0">
@@ -44,5 +45,6 @@
   <joint name="laser_joint0" type="fixed">
     <axis xyz="0 1 0"/>
-    <origin xyz="0 0 0.4" rpy="0 0 0"/>
+    <!-- MUDAR INCLINACAO DO PRIMEIRO AQUI -->
+    <origin xyz="0 0 0.9" rpy="0 0.0777 0"/>
     <parent link="base_link"/>
     <child link="laser_link0"/>
@@ -102,5 +104,5 @@
     <child link="laser_link2"/>
   </joint>
-  <!-- hokuyo2 -->
+  <!-- hokuyo3 -->
   <link name="laser_link3">
     <collision>
@@ -129,5 +131,5 @@
     <child link="laser_link3"/>
   </joint>
-  <!-- hokuyo0 -->
+  <!-- hokuyo scan properties -->
   <gazebo reference="laser_link0">
     <sensor type ="gpu_ray" name="hoyuko0">
@@ -138,14 +140,14 @@
         <scan>
           <horizontal>
-            <samples>720</samples>
-            <resolution>1</resolution>
-            <min_angle>-0.741764</min_angle>
-            <max_angle>0.741764</max_angle>
-          </horizontal>
-        </scan>
-        <range>
-          <min>0.10</min>
-          <max>30</max>
-          <resolution>0.1</resolution>
+            <samples>200</samples>
+            <resolution>1</resolution>
+            <min_angle>-0.741764</min_angle>
+            <max_angle>0.741764</max_angle>
+          </horizontal>
+        </scan>
+        <range>
+          <min>1</min>
+          <max>30</max>
+          <resolution>0.01</resolution>
         </range>
       </ray>
@@ -165,12 +167,12 @@
         <scan>
           <horizontal>
-            <samples>720</samples>
-            <resolution>1</resolution>
-            <min_angle>-0.741764</min_angle>
-            <max_angle>0.741764</max_angle>
-          </horizontal>
-        </scan>
-        <range>
-          <min>0.10</min>
+            <samples>200</samples>
+            <resolution>1</resolution>
+            <min_angle>-0.741764</min_angle>
+            <max_angle>0.741764</max_angle>
+          </horizontal>
+        </scan>
+        <range>
+          <min>1</min>
           <max>30</max>
           <resolution>0.01</resolution>
@@ -192,12 +194,12 @@
         <scan>
           <horizontal>
-            <samples>720</samples>
-            <resolution>1</resolution>
-            <min_angle>-0.741764</min_angle>
-            <max_angle>0.741764</max_angle>
-          </horizontal>
-        </scan>
-        <range>
-          <min>0.10</min>
+            <samples>200</samples>
+            <resolution>1</resolution>
+            <min_angle>-0.741764</min_angle>
+            <max_angle>0.741764</max_angle>
+          </horizontal>
+        </scan>
+        <range>
+          <min>1</min>
           <max>30</max>
           <resolution>0.01</resolution>
@@ -219,12 +221,12 @@
         <scan>
           <horizontal>
-            <samples>720</samples>
-            <resolution>1</resolution>
-            <min_angle>-0.741764</min_angle>
-            <max_angle>0.741764</max_angle>
-          </horizontal>
-        </scan>
-        <range>
-          <min>0.10</min>
+            <samples>200</samples>
+            <resolution>1</resolution>
+            <min_angle>-0.741764</min_angle>
+            <max_angle>0.741764</max_angle>
+          </horizontal>
+        </scan>
+        <range>
+          <min>1</min>
           <max>30</max>
           <resolution>0.01</resolution>
@@ -238,5 +240,3 @@
     </sensor>
   </gazebo>
-  <!-- hokuyo1 -->
-  <!-- <gazebo reference="laser_link1"><sensor type ="gpu_ray" name="hoyuko"><pose>0 0 0 0 0 0</pose><visualize>true</visualize><update_rate>20</update_rate><ray><scan><horizontal><samples>720</samples><resolution>1</resolution><min_angle>-0.741764</min_angle><max_angle>0.741764</max_angle></horizontal></scan><range><min>0.10</min><max>30</max><resolution>0.01</resolution></range></ray><plugin name="gpu_laser" filename="libgazebo_ros_gpu_laser.so"><namespace>/s1</namespace><topicName>/scan1</topicName><frameName>laser_link1</frameName></plugin></sensor></gazebo> -->
 </robot>

Commit message: Correção nos referenciais

File: scan_simulator/urdf/atlas2.urdf.xacro (robot description, xacro)
@@ -46,5 +46,5 @@
     <axis xyz="0 1 0"/>
     <!-- MUDAR INCLINACAO DO PRIMEIRO AQUI -->
-    <origin xyz="0 0 0.9" rpy="0 0.0777 0"/>
+    <origin xyz="0 0 0.4" rpy="0 0.0105 0"/>
     <parent link="base_link"/>
     <child link="laser_link0"/>
@@ -133,24 +133,24 @@
   <!-- hokuyo scan properties -->
   <gazebo reference="laser_link0">
-    <sensor type ="gpu_ray" name="hoyuko0">
-      <pose>0 0 0 0 0 0</pose>
-      <visualize>true</visualize>
-      <update_rate>20</update_rate>
-      <ray>
-        <scan>
-          <horizontal>
-            <samples>200</samples>
-            <resolution>1</resolution>
-            <min_angle>-0.741764</min_angle>
-            <max_angle>0.741764</max_angle>
-          </horizontal>
-        </scan>
-        <range>
-          <min>1</min>
-          <max>30</max>
-          <resolution>0.01</resolution>
-        </range>
-      </ray>
-      <plugin name="gpu_laser" filename="libgazebo_ros_gpu_laser.so">
+    <sensor type ="ray" name="hoyuko0">
+      <pose>0 0 0 0 0 0</pose>
+      <visualize>true</visualize>
+      <update_rate>20</update_rate>
+      <ray>
+        <scan>
+          <horizontal>
+            <samples>200</samples>
+            <resolution>1</resolution>
+            <min_angle>-0.741764</min_angle>
+            <max_angle>0.741764</max_angle>
+          </horizontal>
+        </scan>
+        <range>
+          <min>1</min>
+          <max>40</max>
+          <resolution>0.01</resolution>
+        </range>
+      </ray>
+      <plugin name="laser" filename="libgazebo_ros_laser.so">
         <namespace>/s0</namespace>
         <topicName>/scan0</topicName>
@@ -160,24 +160,24 @@
   </gazebo>
   <gazebo reference="laser_link1">
-    <sensor type ="gpu_ray" name="hoyuko1">
-      <pose>0 0 0 0 0 0</pose>
-      <visualize>true</visualize>
-      <update_rate>20</update_rate>
-      <ray>
-        <scan>
-          <horizontal>
-            <samples>200</samples>
-            <resolution>1</resolution>
-            <min_angle>-0.741764</min_angle>
-            <max_angle>0.741764</max_angle>
-          </horizontal>
-        </scan>
-        <range>
-          <min>1</min>
-          <max>30</max>
-          <resolution>0.01</resolution>
-        </range>
-      </ray>
-      <plugin name="gpu_laser" filename="libgazebo_ros_gpu_laser.so">
+    <sensor type ="ray" name="hoyuko1">
+      <pose>0 0 0 0 0 0</pose>
+      <visualize>true</visualize>
+      <update_rate>20</update_rate>
+      <ray>
+        <scan>
+          <horizontal>
+            <samples>200</samples>
+            <resolution>1</resolution>
+            <min_angle>-0.741764</min_angle>
+            <max_angle>0.741764</max_angle>
+          </horizontal>
+        </scan>
+        <range>
+          <min>1</min>
+          <max>40</max>
+          <resolution>0.01</resolution>
+        </range>
+      </ray>
+      <plugin name="laser" filename="libgazebo_ros_laser.so">
         <namespace>/s1</namespace>
         <topicName>/scan1</topicName>
@@ -187,24 +187,24 @@
   </gazebo>
   <gazebo reference="laser_link2">
-    <sensor type ="gpu_ray" name="hoyuko2">
-      <pose>0 0 0 0 0 0</pose>
-      <visualize>true</visualize>
-      <update_rate>20</update_rate>
-      <ray>
-        <scan>
-          <horizontal>
-            <samples>200</samples>
-            <resolution>1</resolution>
-            <min_angle>-0.741764</min_angle>
-            <max_angle>0.741764</max_angle>
-          </horizontal>
-        </scan>
-        <range>
-          <min>1</min>
-          <max>30</max>
-          <resolution>0.01</resolution>
-        </range>
-      </ray>
-      <plugin name="gpu_laser" filename="libgazebo_ros_gpu_laser.so">
+    <sensor type ="ray" name="hoyuko2">
+      <pose>0 0 0 0 0 0</pose>
+      <visualize>true</visualize>
+      <update_rate>20</update_rate>
+      <ray>
+        <scan>
+          <horizontal>
+            <samples>200</samples>
+            <resolution>1</resolution>
+            <min_angle>-0.741764</min_angle>
+            <max_angle>0.741764</max_angle>
+          </horizontal>
+        </scan>
+        <range>
+          <min>1</min>
+          <max>40</max>
+          <resolution>0.01</resolution>
+        </range>
+      </ray>
+      <plugin name="laser" filename="libgazebo_ros_laser.so">
         <namespace>/s2</namespace>
         <topicName>/scan2</topicName>
@@ -214,24 +214,24 @@
   </gazebo>
   <gazebo reference="laser_link3">
-    <sensor type ="gpu_ray" name="hoyuko3">
-      <pose>0 0 0 0 0 0</pose>
-      <visualize>true</visualize>
-      <update_rate>20</update_rate>
-      <ray>
-        <scan>
-          <horizontal>
-            <samples>200</samples>
-            <resolution>1</resolution>
-            <min_angle>-0.741764</min_angle>
-            <max_angle>0.741764</max_angle>
-          </horizontal>
-        </scan>
-        <range>
-          <min>1</min>
-          <max>30</max>
-          <resolution>0.01</resolution>
-        </range>
-      </ray>
-      <plugin name="gpu_laser" filename="libgazebo_ros_gpu_laser.so">
+    <sensor type ="ray" name="hoyuko3">
+      <pose>0 0 0 0 0 0</pose>
+      <visualize>true</visualize>
+      <update_rate>20</update_rate>
+      <ray>
+        <scan>
+          <horizontal>
+            <samples>200</samples>
+            <resolution>1</resolution>
+            <min_angle>-0.741764</min_angle>
+            <max_angle>0.741764</max_angle>
+          </horizontal>
+        </scan>
+        <range>
+          <min>1</min>
+          <max>40</max>
+          <resolution>0.01</resolution>
+        </range>
+      </ray>
+      <plugin name="laser" filename="libgazebo_ros_laser.so">
         <namespace>/s3</namespace>
         <topicName>/scan3</topicName>
